Commit message: Increased speed ig

File: proper_test/urdf/ur3.urdf (robot description, URDF)
Before this commit: robot ur3, 10 links, 9 joints
Joints:
- joint joint1: limit lower=-3.1415 upper=3.1415 effort=3 velocity=0.1 -> lower=-3.1415 upper=3.1415 effort=3 velocity=1
- joint joint2: limit lower=-3.1415 upper=3.1415 effort=3 velocity=0.1 -> lower=-3.1415 upper=3.1415 effort=3 velocity=1
- joint joint3: limit lower=-3.1415 upper=3.1415 effort=3 velocity=0.1 -> lower=-3.1415 upper=3.1415 effort=3 velocity=1
- joint joint4: limit lower=-3.1415 upper=3.1415 effort=3 velocity=0.1 -> lower=-3.1415 upper=3.1415 effort=3 velocity=1
- joint joint5: limit lower=-3.1415 upper=3.1415 effort=3 velocity=0.1 -> lower=-3.1415 upper=3.1415 effort=3 velocity=1
- joint joint6: limit lower=-3.1415 upper=3.1415 effort=3 velocity=0.1 -> lower=-3.1415 upper=3.1415 effort=3 velocity=1
- joint joint8: limit lower=-0.04 upper=0.0 effort=3 velocity=0.1 -> lower=-0.04 upper=0.0 effort=3 velocity=1
- joint joint9: limit lower=0 upper=0.04 effort=3 velocity=0.1 -> lower=0 upper=0.04 effort=3 velocity=1
